Commit message: Initial framework for adding hand to Atlas?
Significant plumbing changes might be needed to make the
controllers happy with this.

File: examples/Atlas/cylinder.urdf (robot description, URDF)
Before this commit: robot cylinder, 2 links, 1 joints
Links:
- link cylinder_2: geometry collision cylinder length=0.25 radius=0.025; visual cylinder length=1.0 radius=0.025
Joints:
- removed joint cylinder_joint

Commit message: Hand mounted to robot, but pathlcp cries

File: examples/Atlas/cylinder.urdf (robot description, URDF)
Before this commit: robot cylinder, 2 links, 0 joints
Joints:
- added joint cylinder_joint: type revolute, parent cylinder_1, child cylinder_2, origin xyz=0 0 0 rpy=0 -0 0, axis 1 0 0, limit lower=-0.8 upper=0.8 effort=130 velocity=12

Commit message: Plumbing for mounting hand to Atlas
Fixed bug in TSRBM that was unpacking / repacking x <-> q;qd
incorrectly; Atlas can now do previous tests with hands attached
in simul. Moving demonstrative code over to a new test, which will
get developed / cleaned up next.

File: examples/Atlas/cylinder.urdf (robot description, URDF)
Before this commit: robot cylinder, 2 links, 1 joints
Links:
- added link cylinder_3, mass 0.5; collision cylinder length=0.1 radius=0.025; visual cylinder length=0.1 radius=0.025
- link cylinder_1: mass 0.1 -> 0.5
- link cylinder_2: mass 0.1 -> 0.5; geometry collision cylinder length=0.1 radius=0.025; visual cylinder length=0.1 radius=0.025
Joints:
- added joint cylinder_joint_2: type revolute, parent cylinder_2, child cylinder_3, origin xyz=0 0 0 rpy=0 0 0, axis 0 0 1, limit lower=-0.8 upper=0.8 effort=130 velocity=12
- joint cylinder_joint: axis 1 0 0 -> 0 0 1; origin xyz=0 0 0 rpy=0 -0 0 -> xyz=0 0 0 rpy=0 0 0
